File: ipad_lcd/ipad_lcd.kicad_pcb (KiCad board)
At the start: 2 copper layers, 45 x 50 mm, 23 parts, among them P1 CONN_8X2, U1 IPAD3_LCD_CONNECTOR, U2 CONN_DISPLAYPORT_SINK

Commit message: Board probably ready
Parts:
- renumbered LED_GND1 to LED_GND, LED_PWR1 to LED_PWR
Routing:
- net (no net): track 16.1 -> 0.00 mm, vias 7 -> 0
- net GND: track 106.6 -> 117.5 mm, vias 2 -> 5
Other:
- board size 45 x 50 mm -> 45 x 48 mm

Commit message: Changed outline width
Parts:
- added H3: P***, 1pin, F.Cu at (166.1, 137.7)
Changed lines of the file:
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@@
     (links 81)
     (no_connects 0)
-    (area 124.874999 91.674999 169.9006 141.829001)
+    (area 124.874499 93.674499 169.9006 141.829001)
     (thickness 1.6)
     (drawings 4)
     (tracks 440)
     (zones 0)
-    (modules 23)
+    (modules 24)
     (nets 31)
   )
@@
     (trace_min 0.1524)
     (segment_width 0.2)
-    (edge_width 0)
+    (edge_width 0.001)
     (via_size 0.4572)
     (via_drill 0.3048)
@@
     (pcb_text_width 0.3)
     (pcb_text_size 1.5 1.5)
-    (mod_edge_width 0.1)
+    (mod_edge_width 0.001)
     (mod_text_size 1 1)
     (mod_text_width 0.15)
-    (pad_size 1.4 1.4)
-    (pad_drill 1.4)
+    (pad_size 4.064 4.064)
+    (pad_drill 3.048)
     (pad_to_mask_clearance 0)
     (aux_axis_origin 0 0)
@@
     )
   )
-  (gr_line (start 124.875 93.675) (end 124.875 141.675) (angle 90) (layer Edge.Cuts))
-  (gr_line (start 169.875 93.675) (end 124.875 93.675) (angle 90) (layer Edge.Cuts))
-  (gr_line (start 169.875 141.675) (end 169.875 93.675) (angle 90) (layer Edge.Cuts))
-  (gr_line (start 124.875 141.675) (end 169.875 141.675) (angle 90) (layer Edge.Cuts))
+  (module 1pin (layer F.Cu)
+    (at 166.125 137.675)
+    (descr "module 1 pin (ou trou mecanique de percage)")
+    (tags DEV)
+    (path 1pin)
+    (fp_text reference H3 (at 0 -3.048) (layer F.SilkS)
+      (effects (font (size 1.016 1.016) (thickness 0.254)))
+    )
+    (fp_text value P*** (at 0 2.794) (layer F.SilkS) hide
+      (effects (font (size 1.016 1.016) (thickness 0.254)))
+    )
+    (fp_circle (center 0 0) (end 0 -2.286) (layer F.SilkS) (width 0.381))
+    (pad 2 thru_hole circle (at 0 0) (size 4.064 4.064) (drill 3.048)
+      (layers *.Cu *.Mask F.SilkS)
+    )
+  )
+  (gr_line (start 124.875 141.675) (end 169.875 141.675) (angle 90) (layer Edge.Cuts) (width 0.001))
+  (gr_line (start 124.875 93.675) (end 124.875 141.675) (angle 90) (layer Edge.Cuts) (width 0.001))
+  (gr_line (start 169.875 93.675) (end 124.875 93.675) (angle 90) (layer Edge.Cuts) (width 0.001))
+  (gr_line (start 169.875 141.675) (end 169.875 93.675) (angle 90) (layer Edge.Cuts) (width 0.001))
   (via (at 134.51 104.5616) (size 0.4572) (layers F.Cu B.Cu) (net 1))
   (segment (start 137.78 105.28) (end 137.18 105.88) (width 0.1524) (layer F.Cu) (net 1))

Commit message: This version sent off to the fab
Other:
- board text added: "3V3 GND"
- board text added: "iPad LCD adapter by emeryth@gmail.com"
Changed lines of the file:
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@@
     (links 81)
     (no_connects 0)
-    (area 124.874499 93.674499 169.9006 141.829001)
+    (area 103.689286 93.674499 169.9006 141.829001)
     (thickness 1.6)
-    (drawings 4)
+    (drawings 6)
     (tracks 440)
     (zones 0)
@@
     (mod_text_size 1 1)
     (mod_text_width 0.15)
-    (pad_size 4.064 4.064)
-    (pad_drill 3.048)
+    (pad_size 2.1 2.1)
+    (pad_drill 1.7)
     (pad_to_mask_clearance 0)
     (aux_axis_origin 0 0)
@@
     (fp_line (start -10.75 -2.5) (end -10.75 12.5) (layer B.SilkS))
     (fp_line (start 3 -2.5) (end -9.5 -2.5) (layer B.SilkS))
-    (pad 22 thru_hole circle (at -10.75 8.45 180) (size 2 2) (drill 1.6)
+    (pad 22 thru_hole circle (at -10.75 8.45 180) (size 2.1 2.1) (drill 1.7)
       (layers *.Cu *.Mask B.SilkS)
     )
@@
       (layers B.Cu B.Paste B.Mask)
     )
-    (pad 21 thru_hole circle (at 5.75 8.45 180) (size 2 2) (drill 1.6)
+    (pad 21 thru_hole circle (at 5.75 8.45 180) (size 2.1 2.1) (drill 1.7)
       (layers *.Cu *.Mask B.SilkS)
     )
@@
     )
   )
+  (gr_text "3V3 GND" (at 158.125 110.675) (layer F.SilkS)
+    (effects (font (size 1.5 1.5) (thickness 0.3)))
+  )
+  (gr_text "iPad LCD adapter by emeryth@gmail.com" (at 127.375 117.675 90) (layer F.SilkS)
+    (effects (font (size 1.5 1.5) (thickness 0.3)))
+  )
   (gr_line (start 124.875 141.675) (end 169.875 141.675) (angle 90) (layer Edge.Cuts) (width 0.001))
