File: kicad/ipad_lcd/ipad_lcd.kicad_pcb (KiCad board)
At the start: 2 copper layers, 45 x 48 mm, 24 parts, among them P1 CONN_8X2, U1 IPAD3_LCD_CONNECTOR, U2 CONN_DISPLAYPORT_SINK

Commit message: Added Kicad design of new PCB. Reorganized the repo.
Parts:
- R1: value R -> 470R
- R10, R11, R12, R13, R14, R15, R4, R5, R6, R7, R8, R9: value R -> 68R
- R2, R3: value R -> 0R
Changed lines of the file:
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@@
     (links 81)
     (no_connects 0)
-    (area 103.689286 93.674499 169.9006 141.829001)
+    (area 124.874499 93.674499 169.875501 141.675501)
     (thickness 1.6)
     (drawings 6)
@@
     (fp_line (start 5.75 -2.5) (end -10.75 -2.5) (layer B.SilkS) (width 0.1))
     (fp_line (start -10.75 -2.5) (end -10.75 12.5) (layer B.SilkS) (width 0.1))
-    (fp_line (start -10.75 -2.5) (end -10.75 12.5) (layer B.SilkS))
-    (fp_line (start 3 -2.5) (end -9.5 -2.5) (layer B.SilkS))
+    (fp_line (start -10.75 -2.5) (end -10.75 12.5) (layer B.SilkS) (width 0.00012))
+    (fp_line (start 3 -2.5) (end -9.5 -2.5) (layer B.SilkS) (width 0.00012))
     (pad 22 thru_hole circle (at -10.75 8.45 180) (size 2.1 2.1) (drill 1.7)
       (layers *.Cu *.Mask B.SilkS)
@@
     (at 164.465 106.045 90)
     (attr smd)
-    (fp_text reference R1 (at 0 -0.3175 90) (layer F.SilkS)
-      (effects (font (size 0.50038 0.50038) (thickness 0.10922)))
-    )
-    (fp_text value R (at 0 0.635 90) (layer F.SilkS)
+    (fp_text reference R1 (at -0.127 -1.397 90) (layer F.SilkS)
+      (effects (font (size 0.50038 0.50038) (thickness 0.10922)))
+    )
+    (fp_text value 470R (at 0 0.635 90) (layer F.SilkS)
       (effects (font (size 0.50038 0.50038) (thickness 0.10922)))
     )
@@
     (at 158.623 118.11)
     (attr smd)
-    (fp_text reference R5 (at 0 -0.3175) (layer F.SilkS)
-      (effects (font (size 0.50038 0.50038) (thickness 0.10922)))
-    )
-    (fp_text value R (at 0 0.381) (layer F.SilkS)
+    (fp_text reference R5 (at -2.413 -0.254) (layer F.SilkS)
+      (effects (font (size 0.50038 0.50038) (thickness 0.10922)))
+    )
+    (fp_text value 68R (at 0 0.381) (layer F.SilkS)
       (effects (font (size 0.50038 0.50038) (thickness 0.10922)))
     )
@@
     (at 158.623 115.57)
     (attr smd)
-    (fp_text reference R4 (at 0 -0.3175) (layer F.SilkS)
-      (effects (font (size 0.50038 0.50038) (thickness 0.10922)))
-    )
-    (fp_text value R (at 0 0.381) (layer F.SilkS)
+    (fp_text reference R4 (at -2.413 -0.254) (layer F.SilkS)
+      (effects (font (size 0.50038 0.50038) (thickness 0.10922)))
+    )
+    (fp_text value 68R (at 0 0.381) (layer F.SilkS)
       (effects (font (size 0.50038 0.50038) (thickness 0.10922)))
     )
@@
     (at 158.623 123.19)
     (attr smd)
-    (fp_text reference R7 (at 0 -0.3175) (layer F.SilkS)
-      (effects (font (size 0.50038 0.50038) (thickness 0.10922)))
-    )
-    (fp_text value R (at 0 0.381) (layer F.SilkS)
+    (fp_text reference R7 (at -2.413 -0.254) (layer F.SilkS)
+      (effects (font (size 0.50038 0.50038) (thickness 0.10922)))
+    )
+    (fp_text value 68R (at 0 0.381) (layer F.SilkS)
       (effects (font (size 0.50038 0.50038) (thickness 0.10922)))
     )
@@
     (at 158.623 120.65)
     (attr smd)
-    (fp_text reference R6 (at 0 -0.3175) (layer F.SilkS)
-      (effects (font (size 0.50038 0.50038) (thickness 0.10922)))
-    )
-    (fp_text value R (at 0 0.381) (layer F.SilkS)
+    (fp_text reference R6 (at -2.413 -0.254) (layer F.SilkS)
+      (effects (font (size 0.50038 0.50038) (thickness 0.10922)))
+    )
+    (fp_text value 68R (at 0 0.381) (layer F.SilkS)
       (effects (font (size 0.50038 0.50038) (thickness 0.10922)))
     )
@@
     (at 158.623 128.27)
     (attr smd)
-    (fp_text reference R9 (at 0 -0.3175) (layer F.SilkS)
-      (effects (font (size 0.50038 0.50038) (thickness 0.10922)))
-    )
-    (fp_text value R (at 0 0.381) (layer F.SilkS)
+    (fp_text reference R9 (at -2.413 -0.254) (layer F.SilkS)
+      (effects (font (size 0.50038 0.50038) (thickness 0.10922)))
+    )
+    (fp_text value 68R (at 0 0.381) (layer F.SilkS)
       (effects (font (size 0.50038 0.50038) (thickness 0.10922)))
     )
@@
     (at 158.623 125.73)
     (attr smd)
-    (fp_text reference R8 (at 0 -0.3175) (layer F.SilkS)
-      (effects (font (size 0.50038 0.50038) (thickness 0.10922)))
-    )
-    (fp_text value R (at 0 0.381) (layer F.SilkS)
+    (fp_text reference R8 (at -2.413 -0.254) (layer F.SilkS)
+      (effects (font (size 0.50038 0.50038) (thickness 0.10922)))
+    )
+    (fp_text value 68R (at 0 0.381) (layer F.SilkS)
       (effects (font (size 0.50038 0.50038) (thickness 0.10922)))
     )
@@
     (at 158.671 118.101)
     (attr smd)
-    (fp_text reference R11 (at 0 0.3175) (layer B.SilkS)
-      (effects (font (size 0.50038 0.50038) (thickness 0.10922)) (justify mirror))
-    )
-    (fp_text value R (at 0 -0.381) (layer B.SilkS)
+    (fp_text reference R11 (at -2.715 0.517) (layer B.SilkS)
+      (effects (font (size 0.50038 0.50038) (thickness 0.10922)) (justify mirror))
+    )
+    (fp_text value 68R (at 0 -0.381) (layer B.SilkS)
       (effects (font (size 0.50038 0.50038) (thickness 0.10922)) (justify mirror))
     )
@@
     (at 158.671 115.561)
     (attr smd)
-    (fp_text reference R10 (at 0 0.3175) (layer B.SilkS)
-      (effects (font (size 0.50038 0.50038) (thickness 0.10922)) (justify mirror))
-    )
-    (fp_text value R (at 0 -0.381) (layer B.SilkS)
+    (fp_text reference R10 (at -2.715 0.517) (layer B.SilkS)
+      (effects (font (size 0.50038 0.50038) (thickness 0.10922)) (justify mirror))
+    )
+    (fp_text value 68R (at 0 -0.381) (layer B.SilkS)
       (effects (font (size 0.50038 0.50038) (thickness 0.10922)) (justify mirror))
     )
@@
     (at 158.671 123.181)
     (attr smd)
-    (fp_text reference R13 (at 0 0.3175) (layer B.SilkS)
-      (effects (font (size 0.50038 0.50038) (thickness 0.10922)) (justify mirror))
-    )
-    (fp_text value R (at 0 -0.381) (layer B.SilkS)
+    (fp_text reference R13 (at -2.715 0.517) (layer B.SilkS)
+      (effects (font (size 0.50038 0.50038) (thickness 0.10922)) (justify mirror))
+    )
+    (fp_text value 68R (at 0 -0.381) (layer B.SilkS)
       (effects (font (size 0.50038 0.50038) (thickness 0.10922)) (justify mirror))
     )
@@
     (at 158.671 120.641)
     (attr smd)
-    (fp_text reference R12 (at 0 0.3175) (layer B.SilkS)
-      (effects (font (size 0.50038 0.50038) (thickness 0.10922)) (justify mirror))
-    )
-    (fp_text value R (at 0 -0.381) (layer B.SilkS)
+    (fp_text reference R12 (at -2.715 0.517) (layer B.SilkS)
+      (effects (font (size 0.50038 0.50038) (thickness 0.10922)) (justify mirror))
+    )
+    (fp_text value 68R (at 0 -0.381) (layer B.SilkS)
       (effects (font (size 0.50038 0.50038) (thickness 0.10922)) (justify mirror))
     )
@@
     (at 158.671 128.261)
     (attr smd)
-    (fp_text reference R15 (at 0 0.3175) (layer B.SilkS)
-      (effects (font (size 0.50038 0.50038) (thickness 0.10922)) (justify mirror))
-    )
-    (fp_text value R (at 0 -0.381) (layer B.SilkS)
+    (fp_text reference R15 (at -2.715 0.517) (layer B.SilkS)
+      (effects (font (size 0.50038 0.50038) (thickness 0.10922)) (justify mirror))
+    )
+    (fp_text value 68R (at 0 -0.381) (layer B.SilkS)
       (effects (font (size 0.50038 0.50038) (thickness 0.10922)) (justify mirror))
     )
@@
     (at 158.671 125.721)
     (attr smd)
-    (fp_text reference R14 (at 0 0.3175) (layer B.SilkS)
-      (effects (font (size 0.50038 0.50038) (thickness 0.10922)) (justify mirror))
-    )
-    (fp_text value R (at 0 -0.381) (layer B.SilkS)
+    (fp_text reference R14 (at -2.715 0.517) (layer B.SilkS)
+      (effects (font (size 0.50038 0.50038) (thickness 0.10922)) (justify mirror))
+    )
+    (fp_text value 68R (at 0 -0.381) (layer B.SilkS)
       (effects (font (size 0.50038 0.50038) (thickness 0.10922)) (justify mirror))
     )
@@
     (at 158.623 113.03)
     (attr smd)
-    (fp_text reference R2 (at 0 -0.3175) (layer F.SilkS)
-      (effects (font (size 0.50038 0.50038) (thickness 0.10922)))
-    )
-    (fp_text value R (at 0 0.381) (layer F.SilkS)
+    (fp_text reference R2 (at -2.413 -0.508) (layer F.SilkS)
+      (effects (font (size 0.50038 0.50038) (thickness 0.10922)))
+    )
+    (fp_text value 0R (at 0 0.381) (layer F.SilkS)
       (effects (font (size 0.50038 0.50038) (thickness 0.10922)))
     )
@@
     (at 158.671 113.021)
     (attr smd)
-    (fp_text reference R3 (at 0 0.3175) (layer B.SilkS)
-      (effects (font (size 0.50038 0.50038) (thickness 0.10922)) (justify mirror))
-    )
-    (fp_text value R (at 0 -0.381) (layer B.SilkS)
-      (effects (font (size 0.50038 0.50038) (thickness 0.10922)) (justify mirror))
-    )
+    (fp_text reference R3 (at -2.461 0.263) (layer B.SilkS)
+      (effects (font (size 0.50038 0.50038) (thickness 0.10922)) (justify mirror))
+    )
+    (fp_text value 0R (at 0 -0.381) (layer B.SilkS)
+      (effects (font (size 0.50038 0.50038) (thickness 0.10922)) (justify mirror))
+    )
